File: 5V_BDC_Module.kicad_sch (KiCad schematic)
At the start: 18 parts, among them J1 Conn_01x10_Pin, J2 Conn_01x10_Pin, J4 Conn_01x10_Pin, U1 TPS54531DDA

Commit message: unbreak schematic
Parts:
- renumbered C6 to C20, R2 to R11
