File: galaxsea_26_pdb.kicad_pcb (KiCad board)
At the start: 2 copper layers, 50 x 50 mm, 29 parts, among them J1 Conn_01x10_Pin, J2 Conn_01x10_Pin, J3 Conn_01x10_Pin, J4 Conn_01x02, J5 Conn_01x02, U1 TPS54531DDA

Commit message: update mounting
Parts:
- removed J3: Conn_01x10_Pin, Connector_PinHeader_2.54mm:PinHeader_1x10_P2.54mm_Vertical
- J1, J2: value Conn_01x10_Pin -> Conn_01x02; footprint Connector_PinHeader_2.54mm:PinHeader_1x10_P2.54mm_Vertical -> Connector_AMASS:AMASS_XT30U-F_1x02_P5.0mm_Vertical
- J4, J5: moved to B.Cu
- moved TP1 25.8 mm to (148.2, 62.0)
- moved TP2 20.5 mm to (159.2, 62.0)
- moved F1 13.8 mm to (131.2, 76.2)
- moved D3 6.97 mm to (143.3, 67.3)
- moved D2 6.97 mm to (137.9, 67.3)
- moved R4 6.97 mm to (137.9, 71.6)
- moved R5 6.97 mm to (143.3, 71.5)
- moved J5 5.18 mm to (169.0, 62.8)
- moved J4 4.80 mm to (130.0, 62.8)
- moved J1 2.83 mm to (130.0, 102.8), turned to 90 degrees
- moved J2 2.83 mm to (170.0, 102.8), turned to 90 degrees
- moved TP3 1.10 mm to (153.7, 62.0), turned to 0 degrees
Connections:
- J1 pad 1: /BDC Module/BDC_VIN -> GND
- J1 pad 2: /BDC Module/BDC_VIN -> GND
- J2 pad 1: /BDC Module/BDC_VOUT -> GND
- J2 pad 2: /BDC Module/BDC_VOUT -> GND
- TP1 pad 1: /BDC Module/BDC_VIN -> /BDC Module/BDC_VIN_Fuse
Routing:
- net /BDC Module/BDC_VIN: track 36.3 -> 8.48 mm
- net /BDC Module/BDC_VIN_Fuse: track 20.3 -> 45.6 mm
- net /BDC Module/BDC_VOUT: track 62.1 -> 51.2 mm

Commit message: Finalize schematic & layout
Parts:
- removed D2, D3: LED, LED_SMD:LED_1206_3216Metric
- removed F1: Fuse_Small, Fuse:Fuse_1206_3216Metric
- removed J4, J5: Conn_01x02, Connector_AMASS:AMASS_XT30U-F_1x02_P5.0mm_Vertical
- removed R4: 620, Resistor_SMD:R_0603_1608Metric
- removed R5: 150/510, Resistor_SMD:R_0603_1608Metric
- added C10: 10u, Capacitor_SMD:C_0805_2012Metric, F.Cu at (140.3, 88.5)
- added H1: M2, MountingHole:MountingHole_2.2mm_M2, F.Cu at (170.0, 102.8)
- added H2: M2, MountingHole:MountingHole_2.2mm_M2, F.Cu at (130.0, 102.8)
- added H3: M2, MountingHole:MountingHole_2.2mm_M2, F.Cu at (130.0, 62.8)
- added H4: M2, MountingHole:MountingHole_2.2mm_M2, F.Cu at (170.0, 62.8)
- D1: footprint Diode_SMD:D_0805_2012Metric -> Diode_SMD:D_SMC
- J1, J2: value Conn_01x02 -> XT-30; footprint Connector_AMASS:AMASS_XT30U-F_1x02_P5.0mm_Vertical -> Connector_AMASS:AMASS_XT60-F_1x02_P7.20mm_Vertical; moved to F.Cu
- L1: value 5.6u/8.2u -> 5.6u; footprint Inductor_SMD:L_APV_ANR4018 -> Inductor_SMD:L_Vishay_IHLP-2525
- R3: value 1.96k/732 -> 1.96k
- moved TP3 37.5 mm to (164.5, 97.9)
- moved J1 23.6 mm to (130.0, 79.2), turned to -90 degrees
- moved J2 23.6 mm to (170.0, 79.2), turned to -90 degrees
- moved TP1 20.8 mm to (130.0, 72.0)
- moved TP2 14.7 mm to (170.0, 72.0)
- moved D1 4.92 mm to (150.0, 83.0)
- moved C8 3.79 mm to (149.5, 76.9)
- moved C9 3.79 mm to (151.7, 76.9)
- moved C7 3.79 mm to (147.4, 76.9)
- moved L1 2.82 mm to (158.7, 78.3)
- moved G*** 1.50 mm to (138.0, 103.0)
- moved R1 0.99 mm to (161.8, 86.7)
- moved R3 0.99 mm to (161.8, 90.8)
- moved C1 0.81 mm to (154.7, 87.5)
Connections:
- C2 pad 1: /BDC Module/BDC_VIN_Fuse -> /BDC Module/BDC_VIN
- C3 pad 1: /BDC Module/BDC_VIN_Fuse -> /BDC Module/BDC_VIN
- J1 pad 2: GND -> /BDC Module/BDC_VIN
- J2 pad 2: GND -> /BDC Module/BDC_VOUT
- TP1 pad 1: /BDC Module/BDC_VIN_Fuse -> /BDC Module/BDC_VIN
- U1 pad 2: /BDC Module/BDC_VIN_Fuse -> /BDC Module/BDC_VIN
Routing:
- net /BDC Module/BDC_VIN_Fuse: track 45.6 -> 0.00 mm
- net /BDC Module/BDC_VIN: track 8.48 -> 28.8 mm
- net /BDC Module/BDC_VOUT: track 51.2 -> 34.7 mm
- net GND: track 2.59 -> 10.6 mm, vias 39 -> 44
- net Net-(D2-A): track 2.12 -> 0.00 mm
- net Net-(D3-A): track 2.05 -> 0.00 mm
- net /BDC Module/_BDC_VSENSE: track 18.4 -> 17.4 mm
- added copper zone on F.Cu, net /BDC Module/BDC_VIN
- removed copper zone on F.Cu, net /BDC Module/BDC_VIN_Fuse
Other:
- board text added: "TPS54531DDA Test Module {dblquote}Stark{dblquote} Nathan Wignall ${CURRENT_DATE}"
- board text removed: "TPS54531DDA Buck Converter Module Nathan Wignall ${CURRENT_DATE}"
