File: productionBDC.kicad_sch (KiCad schematic)
At the start: 7 parts, among them J10 Screw Terminal Block, J11 Conn_01x36, J15 XT-30, J16 XT-30, J8 JST-XH, J9 XT-30

Commit message: Prepare for PDR
Parts:
- removed J10: Screw Terminal Block, TerminalBlock:TerminalBlock_Altech_AK300-3_P5.00mm, symbol Connector_Generic:Conn_01x03
- removed J16, J9: XT-30, Connector_AMASS:AMASS_XT30UPB-F_1x02_P5.0mm_Vertical, symbol Connector_Generic:Conn_01x02
- removed J8: JST-XH, Connector_JST:JST_XH_B3B-XH-AM_1x03_P2.50mm_Vertical, symbol Connector_Generic:Conn_01x03
- added J13, J8: XT-30, Connector_AMASS:AMASS_XT30UPB-F_1x02_P5.0mm_Vertical, symbol Connector_Generic:Conn_01x02
Connections:
- net GND: now also J13.1 (Pin_1), J8.1 (Pin_1)
- net VOUT: now also J13.2 (Pin_2), J8.2 (Pin_2)
Other:
- moved on the sheet: J15
